Commit message: Initial commit

File: widowx_arm_description/urdf/widowx.urdf.xacro (robot description, xacro)
@@ -1,6 +1,6 @@
 <?xml version="1.0" encoding="UTF-8"?>
 <robot xmlns:xacro="http://ros.org/wiki/xacro">
-   <property name="M_SCALE" value="0.001"/>
-   <property name="M_PI" value="3.14159"/>
+   <xacro:property name="M_SCALE" value="0.001"/>
+   <xacro:property name="M_PI" value="3.14159"/>
    <xacro:include filename="$(find widowx_arm_description)/urdf/common_materials.xacro" />
    <!--link name="plate_top_link"/-->
@@ -53,15 +53,14 @@
       <link name="${prefix}biceps_link">
          <visual>
-			      <origin xyz="${M_SCALE*48.25} 0 ${M_SCALE*140}" rpy="0 0 0" />
-            <!--origin xyz="0 0 0" rpy="0 0 0" /-->
-            <geometry>
-               <mesh filename="package://widowx_arm_description/meshes/biceps_link.stl" />
-            </geometry>
-            <xacro:material_black />
-         </visual>
-         <collision>
-            <origin xyz="0 0 0" rpy="0 0 0" />
-            <geometry>
-               <mesh filename="package://widowx_arm_description/meshes/biceps_link.stl" />
+            <origin xyz="0 0 0" rpy="0 0 0" />
+            <geometry>
+               <mesh filename="package://widowx_arm_description/meshes/biceps_link.new.stl" />
+            </geometry>
+            <xacro:material_black />
+         </visual>
+         <collision>
+            <origin xyz="0 0 0" rpy="0 0 0" />
+            <geometry>
+               <mesh filename="package://widowx_arm_description/meshes/biceps_link.new.stl" />
             </geometry>
          </collision>
@@ -74,8 +73,7 @@
       <link name="${prefix}forearm_link">
          <visual>
-			      <origin xyz="0 0 ${M_SCALE*142.03}" rpy="0 0 0" />
-			<!--origin xyz="0 0 0" rpy="0 0 0" /-->
-            <geometry>
-               <mesh filename="package://widowx_arm_description/meshes/forearm_link.stl"/>
+            <origin xyz="0 0 0" rpy="0 0 0" />
+            <geometry>
+               <mesh filename="package://widowx_arm_description/meshes/forearm_link.new.stl"/>
             </geometry>
            <xacro:material_black />
@@ -84,5 +82,5 @@
             <origin xyz="0 0 0" rpy="0 0 0" />
             <geometry>
-               <mesh filename="package://widowx_arm_description/meshes/forearm_link.stl"/>
+               <mesh filename="package://widowx_arm_description/meshes/forearm_link.new.stl"/>
             </geometry>
          </collision>
@@ -115,23 +113,23 @@
       <link name="${prefix}wrist_2_link">
          <visual>
-            <origin xyz="0 0 ${M_SCALE*43}" rpy="0 0 0" />
-            <geometry>
-               <mesh filename="package://widowx_arm_description/meshes/wrist_2_link.stl"/>
-            </geometry>
-            <xacro:material_black />
-         </visual>
-         <collision>
-            <origin xyz="0 0 0" rpy="0 0 0" />
-            <geometry>
-               <mesh filename="package://widowx_arm_description/meshes/wrist_2_link.stl"/>
-            </geometry>
-         </collision>
-         <inertial>
-            <origin xyz="0 0 0" rpy="0 0 0" />
-            <mass value="1" />
-            <inertia ixx="1.0" ixy="0.0" ixz="0.0" iyy="1.0" iyz="0.0" izz="1.0" />
-         </inertial>
-      </link>
-      <link name="${prefix}gripper_rail_link">
+            <origin xyz="0 0 0" rpy="0 0 0" />
+            <geometry>
+               <mesh filename="package://widowx_arm_description/meshes/wrist_2_link.new.stl"/>
+            </geometry>
+            <xacro:material_black />
+         </visual>
+         <collision>
+            <origin xyz="0 0 0" rpy="0 0 0" />
+            <geometry>
+               <mesh filename="package://widowx_arm_description/meshes/wrist_2_link.new.stl"/>
+            </geometry>
+         </collision>
+         <inertial>
+            <origin xyz="0 0 0" rpy="0 0 0" />
+            <mass value="1" />
+            <inertia ixx="1.0" ixy="0.0" ixz="0.0" iyy="1.0" iyz="0.0" izz="1.0" />
+         </inertial>
+      </link>
+      <!--link name="${prefix}gripper_rail_link">
          <visual>
             <origin xyz="0 0 0" rpy="0 0 1.57" />
@@ -152,8 +150,8 @@
             <inertia ixx="1.0" ixy="0.0" ixz="0.0" iyy="1.0" iyz="0.0" izz="1.0" />
          </inertial>
-      </link>
-      <link name="${prefix}gripper_aux_link">
-      </link>
-      <link name="${prefix}gripper_1_link">
+      </link-->
+      <!--link name="${prefix}gripper_aux_link">
+      </link-->
+      <!--link name="${prefix}gripper_1_link">
          <visual>
             <origin xyz="0 -0.0007 0" rpy="0 0 1.57" />
@@ -194,8 +192,8 @@
             <inertia ixx="1.0" ixy="0.0" ixz="0.0" iyy="1.0" iyz="0.0" izz="1.0" />
          </inertial>
-      </link>
+      </link-->
       <!-- joints -->
       <joint name="${prefix}arm_base_joint" type="fixed">
-         <insert_block name="origin" />
+         <xacro:insert_block name="origin" />
          <parent link="${parent}" />
          <child link="${prefix}arm_base_link"/>
@@ -206,5 +204,5 @@
          <child link="${prefix}shoulder_link" />
          <axis xyz="0 0 1" />
-         <limit lower="-2.617" upper="2.617" effort="0" velocity="0.785" />
+         <limit lower="-2.617" upper="2.617" effort="6" velocity="0.785" />
       </joint>
       <joint name="${prefix}joint_2" type="revolute">
@@ -214,5 +212,5 @@
          <child link="${prefix}biceps_link" />
          <axis xyz="0 1 0" />
-         <limit lower="-1.571" upper="1.571" effort="0" velocity="1.571" />
+         <limit lower="-1.571" upper="1.571" effort="6" velocity="1.571" />
       </joint>
       <joint name="${prefix}joint_3" type="revolute">
@@ -221,5 +219,5 @@
          <child link="${prefix}forearm_link" />
          <axis xyz="0 1 0" />
-         <limit lower="-1.571" upper="1.571" effort="0" velocity="1.571" />
+         <limit lower="-1.571" upper="1.571" effort="6" velocity="1.571" />
       </joint>
       <joint name="${prefix}joint_4" type="revolute">
@@ -228,5 +226,5 @@
          <child link="${prefix}wrist_1_link" />
          <axis xyz="0 1 0" />
-         <limit lower="-1.745" upper="1.745" effort="0" velocity="1.571" />
+         <limit lower="-1.745" upper="1.745" effort="6" velocity="1.571" />
       </joint>
       <joint name="${prefix}joint_5" type="revolute">
@@ -235,26 +233,26 @@
          <child link="${prefix}wrist_2_link" />
          <axis xyz="0 0 1" />
-         <limit lower="-2.617" upper="2.617" effort="0" velocity="1.571" />
-      </joint>
-      <joint name="${prefix}joint_6" type="fixed">
+         <limit lower="-2.617" upper="2.617" effort="6" velocity="1.571" />
+      </joint>
+      <!--joint name="${prefix}joint_6" type="fixed">
          <origin xyz = "0 0 ${M_SCALE*43}" rpy="0 0 0" />
          <parent link="${prefix}wrist_2_link" />
          <child link="${prefix}gripper_rail_link" />
          <axis xyz="0 0 1" />
-         <limit lower="-0.31" upper="0.1" effort="0" velocity="0.5" />
-      </joint>
-      <joint name="${prefix}gripper_revolute_joint" type="revolute">
-         <origin xyz = "0 0 0" rpy="0 0 0" />
-         <parent link="${prefix}gripper_rail_link" />
+         <limit lower="-0.31" upper="0.1" effort="6" velocity="0.5" />
+      </joint-->
+      <!--joint name="${prefix}gripper_revolute_joint" type="revolute">
+         <origin xyz = "0 0 0.065" rpy="0 0 0" />
+         <parent link="${prefix}wrist_2_link" />
          <child link="${prefix}gripper_aux_link" />
          <axis xyz="0 0 1" />
-         <limit lower="0" upper="2.6" effort="0" velocity="0.5" />
-      </joint>
-      <joint name="${prefix}gripper_prismatic_joint_1" type="prismatic">
+         <limit lower="-2.6" upper="2.6" effort="6" velocity="0.5" />
+      </joint-->
+      <!--joint name="${prefix}gripper_prismatic_joint_1" type="prismatic">
          <origin xyz="0 0 0" rpy="0 0 0" />
          <parent link="${prefix}gripper_rail_link" />
          <child link="${prefix}gripper_1_link" />
          <axis xyz="0 -1 0" />
-         <limit lower="0" upper="0.027" effort="0" velocity="0.5" />
+         <limit lower="0" upper="0.027" effort="6" velocity="0.5" />
       </joint>
       <joint name="${prefix}gripper_prismatic_joint_2" type="prismatic">
@@ -264,6 +262,16 @@
          <mimic joint="${prefix}gripper_prismatic_joint_1" />
          <axis xyz="0 1 0" />
-         <limit lower="0" upper="0.027" effort="0" velocity="0.5" />
-      </joint>
+         <limit lower="0" upper="0.027" effort="6" velocity="0.5" />
+      </joint-->
+      <!-- gripper -->
+  <xacro:include filename="$(find widowx_arm_description)/urdf/widowx_gripper.xacro"/>
+  <!--link name="gripper_link"/>
+    <joint name="gripper_link_joint" type="revolute">
+      <origin xyz="0 0 0.110" rpy="0 0 0"/>
+      <parent link="${prefix}wrist_1_link" />
+      <child link="gripper_link"/>
+      <limit effort="6" velocity="1" lower="-3.14" upper="3.14"/>
+      <axis xyz="1 0 0"/>
+    </joint-->
    </xacro:macro>
   <transmission name="tran1">

Commit message: fixed grasping

File: widowx_arm_description/urdf/widowx.urdf.xacro (robot description, xacro)
@@ -213,5 +213,5 @@
          <child link="${prefix}shoulder_link" />
          <axis xyz="0 0 1" />
-         <limit lower="-2.617" upper="2.617" effort="60" velocity="0.785" />
+         <limit lower="-2.617" upper="2.617" effort="1000" velocity="0.785" />
       </joint>
       <joint name="${prefix}joint_2" type="revolute">
@@ -221,5 +221,5 @@
          <child link="${prefix}biceps_link" />
          <axis xyz="0 1 0" />
-         <limit lower="-1.571" upper="1.571" effort="60" velocity="1.571" />
+         <limit lower="-1.571" upper="1.571" effort="1000" velocity="1.571" />
       </joint>
       <joint name="${prefix}joint_3" type="revolute">
@@ -228,5 +228,5 @@
          <child link="${prefix}forearm_link" />
          <axis xyz="0 1 0" />
-         <limit lower="-1.571" upper="1.571" effort="60" velocity="1.571" />
+         <limit lower="-1.571" upper="1.571" effort="1000" velocity="1.571" />
       </joint>
       <joint name="${prefix}joint_4" type="revolute">
@@ -235,5 +235,5 @@
          <child link="${prefix}wrist_1_link" />
          <axis xyz="0 1 0" />
-         <limit lower="-1.745" upper="1.745" effort="60" velocity="1.571" />
+         <limit lower="-1.745" upper="1.745" effort="1000" velocity="1.571" />
       </joint>
       <joint name="${prefix}joint_5" type="revolute">
@@ -242,5 +242,5 @@
          <child link="${prefix}wrist_2_link" />
          <axis xyz="0 0 1" />
-         <limit lower="-2.617" upper="2.617" effort="60" velocity="1.571" />
+         <limit lower="-2.617" upper="2.617" effort="1000" velocity="1.571" />
       </joint>
       <!--joint name="${prefix}joint_6" type="fixed">
@@ -287,8 +287,8 @@
     <type>transmission_interface/SimpleTransmission</type>
     <joint name="joint_1">
-      <hardwareInterface>PositionJointInterface</hardwareInterface>
+      <hardwareInterface>EffortJointInterface</hardwareInterface>
     </joint>
     <actuator name="motor1">
-      <hardwareInterface>PositionJointInterface</hardwareInterface>
+      <hardwareInterface>EffortJointInterface</hardwareInterface>
       <mechanicalReduction>1</mechanicalReduction>
     </actuator>
@@ -297,8 +297,8 @@
     <type>transmission_interface/SimpleTransmission</type>
     <joint name="joint_2">
-      <hardwareInterface>PositionJointInterface</hardwareInterface>
+      <hardwareInterface>EffortJointInterface</hardwareInterface>
     </joint>
     <actuator name="motor2">
-      <hardwareInterface>PositionJointInterface</hardwareInterface>
+      <hardwareInterface>EffortJointInterface</hardwareInterface>
       <mechanicalReduction>1</mechanicalReduction>
     </actuator>
@@ -307,8 +307,8 @@
     <type>transmission_interface/SimpleTransmission</type>
     <joint name="joint_3">
-      <hardwareInterface>PositionJointInterface</hardwareInterface>
+      <hardwareInterface>EffortJointInterface</hardwareInterface>
     </joint>
     <actuator name="motor3">
-      <hardwareInterface>PositionJointInterface</hardwareInterface>
+      <hardwareInterface>EffortJointInterface</hardwareInterface>
       <mechanicalReduction>1</mechanicalReduction>
     </actuator>
@@ -317,8 +317,8 @@
     <type>transmission_interface/SimpleTransmission</type>
     <joint name="joint_4">
-      <hardwareInterface>PositionJointInterface</hardwareInterface>
+      <hardwareInterface>EffortJointInterface</hardwareInterface>
     </joint>
     <actuator name="motor4">
-      <hardwareInterface>PositionJointInterface</hardwareInterface>
+      <hardwareInterface>EffortJointInterface</hardwareInterface>
       <mechanicalReduction>1</mechanicalReduction>
     </actuator>
@@ -326,9 +326,9 @@
  <transmission name="tran5">
    <joint name="joint_5">
-     <hardwareInterface>PositionJointInterface</hardwareInterface>
+     <hardwareInterface>EffortJointInterface</hardwareInterface>
    </joint>
     <type>transmission_interface/SimpleTransmission</type>
     <actuator name="motor5">
-      <hardwareInterface>PositionJointInterface</hardwareInterface>
+      <hardwareInterface>EffortJointInterface</hardwareInterface>
       <mechanicalReduction>1</mechanicalReduction>
     </actuator>
@@ -337,8 +337,8 @@
     <type>transmission_interface/SimpleTransmission</type>
     <joint name="gripper_joint_1">
-      <hardwareInterface>PositionJointInterface</hardwareInterface>
+      <hardwareInterface>EffortJointInterface</hardwareInterface>
     </joint>
     <actuator name="motor6">
-      <hardwareInterface>PositionJointInterface</hardwareInterface>
+      <hardwareInterface>EffortJointInterface</hardwareInterface>
       <mechanicalReduction>1</mechanicalReduction>
     </actuator>
@@ -347,8 +347,8 @@
      <type>transmission_interface/SimpleTransmission</type>
      <joint name="gripper_joint_2">
-       <hardwareInterface>PositionJointInterface</hardwareInterface>
+       <hardwareInterface>EffortJointInterface</hardwareInterface>
      </joint>
      <actuator name="motor7">
-       <hardwareInterface>PositionJointInterface</hardwareInterface>
+       <hardwareInterface>EffortJointInterface</hardwareInterface>
        <mechanicalReduction>1</mechanicalReduction>
      </actuator>

File: widowx_arm_description/urdf/widowx_gripper.xacro (robot description, xacro)
@@ -17,5 +17,5 @@
       <inertial>
          <origin xyz="0 0 0" rpy="0 0 0" />
-         <mass value="1" />
+         <mass value="0.1" />
          <inertia ixx="1.0" ixy="0.0" ixz="0.0" iyy="1.0" iyz="0.0" izz="1.0" />
       </inertial>
@@ -56,6 +56,6 @@
           <friction>
             <ode>
-              <mu>1e10</mu>
-              <mu2>1e10</mu2>
+              <mu>1</mu>
+              <mu2>1</mu2>
               <fdir1>0.000000 0.000000 1.000000</fdir1>
             </ode>
@@ -71,5 +71,5 @@
       <inertial>
          <origin xyz="0 0 0" rpy="0 0 0" />
-         <mass value="1" />
+         <mass value="0.1" />
          <inertia ixx="1.0" ixy="0.0" ixz="0.0" iyy="1.0" iyz="0.0" izz="1.0" />
       </inertial>
@@ -108,6 +108,6 @@
           <friction>
             <ode>
-              <mu>1e10</mu>
-              <mu2>1e10</mu2>
+              <mu>1</mu>
+              <mu2>1</mu2>
               <fdir1>0.000000 0.000000 1.000000</fdir1>
             </ode>
@@ -123,5 +123,5 @@
       <inertial>
          <origin xyz="0 0 0" rpy="0 0 0" />
-         <mass value="1" />
+         <mass value="0.1" />
          <inertia ixx="1.0" ixy="0.0" ixz="0.0" iyy="1.0" iyz="0.0" izz="1.0" />
       </inertial>
@@ -138,5 +138,5 @@
       <child link="${prefix}gripper_1_link" />
       <axis xyz="0 -1 0" />
-      <limit lower="0.002" upper="0.031" effort="6" velocity="0.5" />
+      <limit lower="0.002" upper="0.031" effort="1000" velocity="0.5" />
    </joint>
    <joint name="${prefix}gripper_joint_2" type="prismatic">
@@ -145,5 +145,5 @@
       <child link="${prefix}gripper_2_link" />
       <axis xyz="0 1 0" />
-      <limit lower="0.002" upper="0.031" effort="6" velocity="0.5" />
+      <limit lower="0.002" upper="0.031" effort="1000" velocity="0.5" />
    </joint>
 </robot>
