Commit message: added gazebo simulation capability

File: widowx_arm_description/robots/widowx_arm.urdf.xacro (robot description, xacro)
@@ -10,5 +10,17 @@
 		</visual>
 	</link>
-	<xacro:widowx_arm parent="base_footprint" prefix="">
+	<link name="world">
+		<visual>
+			<origin xyz="0 0 0" rpy="0 0 0"/>
+			<geometry>
+				<box size="0.001 0.001 0.001" />
+			</geometry>
+		</visual>
+	</link>
+	<joint name="fixed" type="fixed">
+    <parent link="world"/>
+    <child link="base_footprint"/>
+  </joint>
+	<xacro:widowx_arm parent="world" prefix="">
 		<origin xyz="0.0 0.0 0.0" rpy="0.0 0.0 0.0"/>
 	</xacro:widowx_arm>

File: widowx_arm_description/urdf/widowx.urdf.xacro (robot description, xacro)
@@ -9,6 +9,15 @@
       <child link="ph_base_link" />
    </joint-->
+   <!-- Import all Gazebo-customization elements, including Gazebo colors -->
+  <xacro:include filename="$(find widowx_arm_description)/urdf/widowx.gazebo" />
+  <gazebo>
+  <plugin name="ros_control" filename="libgazebo_ros_control.so">
+    <!--robotNamespace>/</robotNamespace-->
+    <!--robotSimType>gazebo_ros_control/DefaultRobotHWSim</robotSimType-->
+  </plugin>
+  </gazebo>
    <xacro:macro name="widowx_arm" params="parent prefix *origin">
       <!-- links -->
+      <!-- Used for fixing robot to Gazebo 'base_link' -->
       <link name="${prefix}arm_base_link">
          <visual>
@@ -204,5 +213,5 @@
          <child link="${prefix}shoulder_link" />
          <axis xyz="0 0 1" />
-         <limit lower="-2.617" upper="2.617" effort="6" velocity="0.785" />
+         <limit lower="-2.617" upper="2.617" effort="60" velocity="0.785" />
       </joint>
       <joint name="${prefix}joint_2" type="revolute">
@@ -212,5 +221,5 @@
          <child link="${prefix}biceps_link" />
          <axis xyz="0 1 0" />
-         <limit lower="-1.571" upper="1.571" effort="6" velocity="1.571" />
+         <limit lower="-1.571" upper="1.571" effort="60" velocity="1.571" />
       </joint>
       <joint name="${prefix}joint_3" type="revolute">
@@ -219,5 +228,5 @@
          <child link="${prefix}forearm_link" />
          <axis xyz="0 1 0" />
-         <limit lower="-1.571" upper="1.571" effort="6" velocity="1.571" />
+         <limit lower="-1.571" upper="1.571" effort="60" velocity="1.571" />
       </joint>
       <joint name="${prefix}joint_4" type="revolute">
@@ -226,5 +235,5 @@
          <child link="${prefix}wrist_1_link" />
          <axis xyz="0 1 0" />
-         <limit lower="-1.745" upper="1.745" effort="6" velocity="1.571" />
+         <limit lower="-1.745" upper="1.745" effort="60" velocity="1.571" />
       </joint>
       <joint name="${prefix}joint_5" type="revolute">
@@ -233,5 +242,5 @@
          <child link="${prefix}wrist_2_link" />
          <axis xyz="0 0 1" />
-         <limit lower="-2.617" upper="2.617" effort="6" velocity="1.571" />
+         <limit lower="-2.617" upper="2.617" effort="60" velocity="1.571" />
       </joint>
       <!--joint name="${prefix}joint_6" type="fixed">
@@ -240,5 +249,5 @@
          <child link="${prefix}gripper_rail_link" />
          <axis xyz="0 0 1" />
-         <limit lower="-0.31" upper="0.1" effort="6" velocity="0.5" />
+         <limit lower="-0.31" upper="0.1" effort="60" velocity="0.5" />
       </joint-->
       <!--joint name="${prefix}gripper_revolute_joint" type="revolute">
@@ -247,5 +256,5 @@
          <child link="${prefix}gripper_aux_link" />
          <axis xyz="0 0 1" />
-         <limit lower="-2.6" upper="2.6" effort="6" velocity="0.5" />
+         <limit lower="-2.6" upper="2.6" effort="60" velocity="0.5" />
       </joint-->
       <!--joint name="${prefix}gripper_prismatic_joint_1" type="prismatic">
@@ -254,5 +263,5 @@
          <child link="${prefix}gripper_1_link" />
          <axis xyz="0 -1 0" />
-         <limit lower="0" upper="0.027" effort="6" velocity="0.5" />
+         <limit lower="0" upper="0.027" effort="60" velocity="0.5" />
       </joint>
       <joint name="${prefix}gripper_prismatic_joint_2" type="prismatic">
@@ -262,5 +271,5 @@
          <mimic joint="${prefix}gripper_prismatic_joint_1" />
          <axis xyz="0 1 0" />
-         <limit lower="0" upper="0.027" effort="6" velocity="0.5" />
+         <limit lower="0" upper="0.027" effort="60" velocity="0.5" />
       </joint-->
       <!-- gripper -->
@@ -271,5 +280,5 @@
       <parent link="${prefix}wrist_1_link" />
       <child link="gripper_link"/>
-      <limit effort="6" velocity="1" lower="-3.14" upper="3.14"/>
+      <limit effort="60" velocity="1" lower="-3.14" upper="3.14"/>
       <axis xyz="1 0 0"/>
     </joint-->
@@ -277,7 +286,9 @@
   <transmission name="tran1">
     <type>transmission_interface/SimpleTransmission</type>
-    <joint name="joint_1"/>
+    <joint name="joint_1">
+      <hardwareInterface>PositionJointInterface</hardwareInterface>
+    </joint>
     <actuator name="motor1">
-      <hardwareInterface>EffortJointInterface</hardwareInterface>
+      <hardwareInterface>PositionJointInterface</hardwareInterface>
       <mechanicalReduction>1</mechanicalReduction>
     </actuator>
@@ -285,7 +296,9 @@
  <transmission name="tran2">
     <type>transmission_interface/SimpleTransmission</type>
-    <joint name="joint_2"/>
+    <joint name="joint_2">
+      <hardwareInterface>PositionJointInterface</hardwareInterface>
+    </joint>
     <actuator name="motor2">
-      <hardwareInterface>EffortJointInterface</hardwareInterface>
+      <hardwareInterface>PositionJointInterface</hardwareInterface>
       <mechanicalReduction>1</mechanicalReduction>
     </actuator>
@@ -293,7 +306,9 @@
  <transmission name="tran3">
     <type>transmission_interface/SimpleTransmission</type>
-    <joint name="joint_3"/>
+    <joint name="joint_3">
+      <hardwareInterface>PositionJointInterface</hardwareInterface>
+    </joint>
     <actuator name="motor3">
-      <hardwareInterface>EffortJointInterface</hardwareInterface>
+      <hardwareInterface>PositionJointInterface</hardwareInterface>
       <mechanicalReduction>1</mechanicalReduction>
     </actuator>
@@ -301,15 +316,19 @@
  <transmission name="tran4">
     <type>transmission_interface/SimpleTransmission</type>
-    <joint name="joint_4"/>
+    <joint name="joint_4">
+      <hardwareInterface>PositionJointInterface</hardwareInterface>
+    </joint>
     <actuator name="motor4">
-      <hardwareInterface>EffortJointInterface</hardwareInterface>
+      <hardwareInterface>PositionJointInterface</hardwareInterface>
       <mechanicalReduction>1</mechanicalReduction>
     </actuator>
   </transmission>
  <transmission name="tran5">
-    <type>transmission_interface/SimpleTransmission</type>
-    <joint name="joint_6"/>
+   <joint name="joint_5">
+     <hardwareInterface>PositionJointInterface</hardwareInterface>
+   </joint>
+    <type>transmission_interface/SimpleTransmission</type>
     <actuator name="motor5">
-      <hardwareInterface>EffortJointInterface</hardwareInterface>
+      <hardwareInterface>PositionJointInterface</hardwareInterface>
       <mechanicalReduction>1</mechanicalReduction>
     </actuator>
@@ -317,9 +336,21 @@
  <transmission name="tran6">
     <type>transmission_interface/SimpleTransmission</type>
-    <joint name="gripper_prismatic_joint_1"/>
+    <joint name="gripper_joint_1">
+      <hardwareInterface>PositionJointInterface</hardwareInterface>
+    </joint>
     <actuator name="motor6">
-      <hardwareInterface>EffortJointInterface</hardwareInterface>
-      <mechanicalReduction>1</mechanicalReduction>
-    </actuator>
-  </transmission>
+      <hardwareInterface>PositionJointInterface</hardwareInterface>
+      <mechanicalReduction>1</mechanicalReduction>
+    </actuator>
+  </transmission>
+  <transmission name="tran7">
+     <type>transmission_interface/SimpleTransmission</type>
+     <joint name="gripper_joint_2">
+       <hardwareInterface>PositionJointInterface</hardwareInterface>
+     </joint>
+     <actuator name="motor7">
+       <hardwareInterface>PositionJointInterface</hardwareInterface>
+       <mechanicalReduction>1</mechanicalReduction>
+     </actuator>
+   </transmission>
 </robot>

File: widowx_arm_description/urdf/widowx_gripper.xacro (robot description, xacro)
@@ -69,18 +69,17 @@
       <axis xyz="0 0 1" />
    </joint>
-   <joint name="${prefix}gripper_joint" type="prismatic">
+   <joint name="${prefix}gripper_joint_1" type="prismatic">
       <origin xyz="0 0 0" rpy="0 0 0" />
       <parent link="${prefix}gripper_rail_link" />
       <child link="${prefix}gripper_1_link" />
       <axis xyz="0 -1 0" />
-      <limit lower="0.002" upper="0.031" effort="0" velocity="0.5" />
+      <limit lower="0.002" upper="0.031" effort="6" velocity="0.5" />
    </joint>
-   <joint name="${prefix}gripper_prismatic_joint_2" type="prismatic">
+   <joint name="${prefix}gripper_joint_2" type="prismatic">
       <origin xyz="0 0 0" rpy="0 0 0" />
       <parent link="${prefix}gripper_rail_link" />
       <child link="${prefix}gripper_2_link" />
-      <mimic joint="${prefix}gripper_joint" />
       <axis xyz="0 1 0" />
-      <limit lower="0.002" upper="0.031" effort="0" velocity="0.5" />
+      <limit lower="0.002" upper="0.031" effort="6" velocity="0.5" />
    </joint>
 </robot>
